File: bin_clock_2.kicad_pcb (KiCad board)
At the start: 2 copper layers, 190 x 110 mm, 54 parts, among them J1 bat, J2 power, J3 uart, J4 swd, SW1 SW_Push, SW2 SW_Push, SW3 SW_Push, SW4 SW_Push, SW5 SW_Push, U1 STM32F103C8Tx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

Commit message: done
Parts:
- removed J1: bat, Pin_Headers:Pin_Header_Straight_1x02_Pitch2.54mm
- removed R13: v1R, Resistors_SMD:R_0603_HandSoldering
- removed R14: v2R, Resistors_SMD:R_0603_HandSoldering
- added BT1: cr2032, Battery_Holders:BS-7_CR2032, F.Cu at (132.3, 93.9)
- U2: value LM1117-ADJ -> LM7805CT; footprint TO_SOT_Packages_SMD:TO-252-2Lead -> TO_SOT_Packages_THT:TO-220_Vertical
- Y1: footprint Crystals:Crystal_C38-LF_d3.0mm_l8.0mm_Vertical -> Crystals:Crystal_HC49-4H_Vertical
- moved J2 20.5 mm to (134.9, 137.7), turned to 180 degrees
- moved U2 18.3 mm to (142.2, 137.9)
- moved C6 10.3 mm to (143.5, 135.1), turned to 0 degrees
- moved Y1 8.63 mm to (110.7, 98.2), turned to 90 degrees
- moved C11 8.56 mm to (146.7, 131.7), turned to 180 degrees
- moved C1 4.95 mm to (115.7, 98.2), turned to 0 degrees
- moved C2 3.59 mm to (115.7, 93.3), turned to 0 degrees
- moved J4 1.14 mm to (143.4, 99.7)
- moved C4 1.02 mm to (121.9, 97.2), turned to 0 degrees
Connections:
- U2 pad 1: Net-(R13-Pad2) -> Net-(C6-Pad1)
- U2 pad 2: +3V3 -> GND
- U2 pad 3: Net-(C6-Pad1) -> +3V3
Routing:
- net +3V3: track 932.0 -> 906.8 mm
- net Net-(C2-Pad1): track 11.6 -> 25.9 mm
- net Net-(R13-Pad2): track 13.8 -> 0.00 mm
- net GND: track 171.0 -> 183.6 mm
- net Net-(C1-Pad1): track 12.0 -> 18.8 mm
- net Net-(D1-Pad1): track 0.00 -> 4.40 mm
- net Net-(C6-Pad1): track 12.6 -> 10.2 mm
- net Net-(C5-Pad2): track 16.6 -> 14.9 mm
- net Net-(BT1-Pad1): track 12.1 -> 10.8 mm
Other:
- board text added: "BIN CLOCK v2 by Alexander Lutsai April 2017"

Commit message: pcb ready
Parts:
- moved REF** 41.2 mm to (100.0, 140.0)
- moved REF** 40.0 mm to (100.0, 60.0)
- moved D1 29.0 mm to (98.2, 125.0)
- moved R1 29.0 mm to (98.4, 120.7)
- moved REF** 20.0 mm to (165.0, 60.0)
- moved REF** 10.0 mm to (230.0, 140.0)
- moved C8 3.26 mm to (134.2, 108.2), turned to 90 degrees
Routing:
- net +3V3: track 906.8 -> 580.5 mm
- net /h2: track 264.5 -> 87.0 mm
- net (no net): track 91.4 -> 0.00 mm
- net /h1: track 142.3 -> 107.2 mm
- net /SEC: track 64.4 -> 32.2 mm
- net /b1: track 222.0 -> 198.4 mm
- net /b2: track 206.4 -> 183.1 mm
- net /b3: track 190.9 -> 167.9 mm
- net /b4: track 173.5 -> 150.7 mm
- net /PM: track 104.8 -> 84.3 mm
- net /h4: track 72.1 -> 67.6 mm
- net GND: track 183.6 -> 181.3 mm, vias 1 -> 0
- net /m8: track 45.2 -> 47.2 mm
- net /m16: track 30.0 -> 31.5 mm
- net /m1: track 104.9 -> 103.5 mm
Other:
- board size 190 x 110 mm -> 150 x 100 mm

Commit message: smallest clock
Parts:
- removed J3: uart, Pin_Headers:Pin_Header_Straight_1x03_Pitch2.54mm
- removed the REF** at (165.0, 60.0)
- removed SW2, SW3: SW_Push, Buttons_Switches_THT:SW_PUSH_SMALL
- REF** (x4): value Pin_Header_Straight_1x01_Pitch2.54mm -> Pin
- moved SW5 77.6 mm to (149.7, 102.0)
- moved REF** 76.2 mm to (157.5, 83.5)
- moved SW4 74.6 mm to (149.7, 111.5)
- moved REF** 73.2 mm to (157.5, 130.0)
- moved R12 71.2 mm to (150.0, 86.5)
- moved D12 70.9 mm to (150.0, 83.5)
- moved R11 69.3 mm to (150.0, 118.0)
- moved D11 69.3 mm to (150.0, 122.0)
- moved R10 58.5 mm to (143.0, 86.5)
- moved D10 57.9 mm to (143.0, 83.5)
- moved R9 56.6 mm to (143.0, 118.0)
- moved D9 56.3 mm to (143.0, 122.0)
- moved D7 44.1 mm to (136.0, 122.0)
- moved R7 44.0 mm to (136.0, 118.0)
- moved R8 43.6 mm to (136.0, 86.5)
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Routing:
- net +3V3: track 580.5 -> 247.3 mm
- net /b1: track 198.4 -> 0.00 mm
- net /b2: track 183.1 -> 0.00 mm
- net /b3: track 167.9 -> 24.5 mm
- net /b4: track 150.7 -> 35.6 mm
- net /m1: track 103.5 -> 31.6 mm
- net /h1: track 107.2 -> 46.1 mm
- net /m2: track 85.0 -> 25.6 mm
- net /m4: track 66.5 -> 19.9 mm
- net /h2: track 87.0 -> 47.1 mm
- net /m8: track 47.2 -> 13.7 mm
- net /h4: track 67.6 -> 43.6 mm
- net /m16: track 31.5 -> 12.7 mm
- net /PM: track 84.3 -> 71.5 mm
- net /SEC: track 32.2 -> 25.5 mm
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Other:
- board size 150 x 100 mm -> 65 x 55 mm
- rule trace_min: 0.2 -> 0.15
- board text added: "BIN CLOCK v3 by Александр Луцай February 2018"
- board text added: "made with love"
- board text added: "С 8 Марта, Катя!"
- board text added: "С 8 Марта, Полин!"
- board text removed: "BIN CLOCK v2 by Alexander Lutsai April 2017"
